File: Conectores_E_S.sch (KiCad schematic (older format))
At the start: 9 parts

Commit message: version preliminar de la etapa de alimentacion
Parts:
- gave numbers to parts that had none: 9
Changed lines of the file:
@@
 LIBS:Sensores
 LIBS:Reles
+LIBS:Reguladores
+LIBS:Transistores
 LIBS:Wifi_PB-cache
 EELAYER 26 0
@@
 $Descr A4 11693 8268
 encoding utf-8
-Sheet 11 11
+Sheet 11 15
 Title ""
 Date "2017-01-15"
@@
 $EndDescr
 $Comp
-L USB_MINI P?
+L USB_MINI P11
 U 1 1 583F8179
 P 1600 2000
-F 0 "P?" V 1175 1924 50  0000 C CNN
+F 0 "P11" V 1175 1924 50  0000 C CNN
 F 1 "USB_MINI" V 1266 1924 50  0000 C CNN
-F 2 "" V 1550 1900 50  0000 C CNN
+F 2 "" V 1550 1900 50  0001 C CNN
 F 3 "" V 1550 1900 50  0000 C CNN
 	1    1600 2000
@@
 $EndComp
 $Comp
-L C C?
+L C C27
 U 1 1 583F8180
 P 2550 2500
-F 0 "C?" H 2665 2546 50  0000 L CNN
+F 0 "C27" H 2665 2546 50  0000 L CNN
 F 1 "0,047n" H 2665 2455 50  0000 L CNN
-F 2 "" H 2588 2350 50  0000 C CNN
+F 2 "" H 2588 2350 50  0001 C CNN
 F 3 "" H 2550 2500 50  0000 C CNN
 	1    2550 2500
@@
 $EndComp
 $Comp
-L C C?
+L C C26
 U 1 1 583F8187
 P 2150 2500
-F 0 "C?" H 2265 2546 50  0000 L CNN
+F 0 "C26" H 2265 2546 50  0000 L CNN
 F 1 "10n" H 2265 2455 50  0000 L CNN
-F 2 "" H 2188 2350 50  0000 C CNN
+F 2 "" H 2188 2350 50  0001 C CNN
 F 3 "" H 2150 2500 50  0000 C CNN
 	1    2150 2500
@@
 $EndComp
 $Comp
-L C C?
+L C C28
 U 1 1 583F818E
 P 3050 2500
-F 0 "C?" H 3165 2546 50  0000 L CNN
+F 0 "C28" H 3165 2546 50  0000 L CNN
 F 1 "0,047n" H 3165 2455 50  0000 L CNN
-F 2 "" H 3088 2350 50  0000 C CNN
+F 2 "" H 3088 2350 50  0001 C CNN
 F 3 "" H 3050 2500 50  0000 C CNN
 	1    3050 2500
@@
 $EndComp
 $Comp
-L Ferrita L?
+L Ferrita L1
 U 1 1 583F8195
 P 2450 1800
-F 0 "L?" V 2243 1800 50  0000 C CNN
+F 0 "L1" V 2243 1800 50  0000 C CNN
 F 1 "Ferrita" V 2334 1800 50  0000 C CNN
-F 2 "" V 2380 1800 50  0000 C CNN
+F 2 "" V 2380 1800 50  0001 C CNN
 F 3 "" H 2450 1800 50  0000 C CNN
 	1    2450 1800
@@
 $EndComp
 $Comp
-L F F?
+L F F1
 U 1 1 583F819C
 P 2900 1800
-F 0 "F?" V 2693 1800 50  0000 C CNN
+F 0 "F1" V 2693 1800 50  0000 C CNN
 F 1 "F" V 2784 1800 50  0000 C CNN
-F 2 "" V 2830 1800 50  0000 C CNN
+F 2 "" V 2830 1800 50  0001 C CNN
 F 3 "" H 2900 1800 50  0000 C CNN
 	1    2900 1800
@@
 $EndComp
 $Comp
-L R R?
+L R R47
 U 1 1 583F81A3
 P 3200 1900
-F 0 "R?" V 3250 1700 50  0000 C CNN
+F 0 "R47" V 3250 1700 50  0000 C CNN
 F 1 "22R" V 3200 1900 50  0000 C CNN
-F 2 "" V 3130 1900 50  0000 C CNN
+F 2 "" V 3130 1900 50  0001 C CNN
 F 3 "" H 3200 1900 50  0000 C CNN
 	1    3200 1900
@@
 $EndComp
 $Comp
-L R R?
+L R R48
 U 1 1 583F81AA
 P 3500 2000
-F 0 "R?" V 3550 1800 50  0000 C CNN
+F 0 "R48" V 3550 1800 50  0000 C CNN
 F 1 "22R" V 3500 2000 50  0000 C CNN
-F 2 "" V 3430 2000 50  0000 C CNN
+F 2 "" V 3430 2000 50  0001 C CNN
 F 3 "" H 3500 2000 50  0000 C CNN
 	1    3500 2000
@@
 	3050 3000 3050 2650
 $Comp
-L GND #PWR022
+L GND #PWR80
 U 1 1 583F81C7
 P 2000 3000
-F 0 "#PWR022" H 2000 2750 50  0001 C CNN
+F 0 "#PWR80" H 2000 2750 50  0001 C CNN
 F 1 "GND" H 2005 2827 50  0000 C CNN
 F 2 "" H 2000 3000 50  0000 C CNN
@@
 $EndComp
 $Comp
-L GND #PWR023
+L GND #PWR81
 U 1 1 583F81CD
 P 2550 3000
-F 0 "#PWR023" H 2550 2750 50  0001 C CNN
+F 0 "#PWR81" H 2550 2750 50  0001 C CNN
 F 1 "GND" H 2555 2827 50  0000 C CNN
 F 2 "" H 2550 3000 50  0000 C CNN
@@
 $EndComp
 $Comp
-L GND #PWR024
+L GND #PWR82
 U 1 1 583F81D3
 P 3050 3000
-F 0 "#PWR024" H 3050 2750 50  0001 C CNN
+F 0 "#PWR82" H 3050 2750 50  0001 C CNN
 F 1 "GND" H 3055 2827 50  0000 C CNN
 F 2 "" H 3050 3000 50  0000 C CNN
@@
 $EndComp
 $Comp
-L D_Schottky_ALT D?
+L D_Schottky_ALT D2
 U 1 1 583F81D9
 P 4200 1800
-F 0 "D?" H 4200 1584 50  0000 C CNN
+F 0 "D2" H 4200 1584 50  0000 C CNN
 F 1 "D_Schottky_ALT" H 4200 1675 50  0000 C CNN
-F 2 "" H 4200 1800 50  0000 C CNN
+F 2 "" H 4200 1800 50  0001 C CNN
 F 3 "" H 4200 1800 50  0000 C CNN
 	1    4200 1800
 	-1   0    0    1
 $EndComp
-Text Label 3500 1800 0    60   ~ 0
-VUSB
 Wire Wire Line
 	4350 1800 4650 1800
@@
 	4650 1800 4650 1600
 $Comp
-L +5V #PWR025
+L +5V #PWR83
 U 1 1 583F81E3
 P 4650 1600
-F 0 "#PWR025" H 4650 1450 50  0001 C CNN
+F 0 "#PWR83" H 4650 1450 50  0001 C CNN
 F 1 "+5V" H 4665 1773 50  0000 C CNN
 F 2 "" H 4650 1600 50  0000 C CNN
@@
 	1    0    0    -1
 $EndComp
+Text GLabel 3450 1250 1    60   Output ~ 0
+VUSB
+Wire Wire Line
+	3450 1250 3450 1800
+Connection ~ 3450 1800
 $EndSCHEMATC
