File: Matriz_Led.sch (KiCad schematic (older format))
At the start: 23 parts, among them Q1 SMBT3904, Q2 SMBT3904, Q3 SMBT3904, Q4 SMBT3904, Q5 SMBT3904

Commit message: version preliminar de la etapa de alimentacion
Parts:
- gave numbers to parts that had none: 6
- renumbered Q1 to Q5, Q2 to Q6, Q3 to Q7, Q4 to Q8, Q5 to Q9, R8 to R21, R9 to R22, R10 to R23, R11 to R24, R12 to R25, R2 to R26, R4 to R27, R6 to R28, R1 to R31, R3 to R32, R5 to R33, R7 to R34
Changed lines of the file:
@@
 LIBS:Sensores
 LIBS:Reles
+LIBS:Reguladores
+LIBS:Transistores
 LIBS:Wifi_PB-cache
 EELAYER 26 0
@@
 $Descr A4 11693 8268
 encoding utf-8
-Sheet 8 11
+Sheet 8 15
 Title ""
 Date "2017-01-15"
@@
 $EndDescr
 $Comp
-L GND #PWR015
+L GND #PWR66
 U 1 1 5793BD55
 P 5100 6550
-F 0 "#PWR015" H 5100 6300 50  0001 C CNN
+F 0 "#PWR66" H 5100 6300 50  0001 C CNN
 F 1 "GND" H 5100 6400 50  0000 C CNN
 F 2 "" H 5100 6550 50  0000 C CNN
@@
 $EndComp
 $Comp
-L R R1
+L R R31
 U 1 1 5793BD61
 P 4250 1300
-F 0 "R1" V 4330 1300 50  0000 C CNN
+F 0 "R31" V 4330 1300 50  0000 C CNN
 F 1 "120" V 4250 1300 50  0000 C CNN
 F 2 "Resistencias:R_0805" V 4180 1300 50  0001 C CNN
@@
 	3400 3600 4400 3600
 $Comp
-L R R2
+L R R26
 U 1 1 5793BE17
 P 3700 1400
-F 0 "R2" V 3780 1400 50  0000 C CNN
+F 0 "R26" V 3780 1400 50  0000 C CNN
 F 1 "120" V 3700 1400 50  0000 C CNN
 F 2 "Resistencias:R_0805" V 3630 1400 50  0001 C CNN
@@
 $EndComp
 $Comp
-L R R4
+L R R27
 U 1 1 5793BE24
 P 3700 1600
-F 0 "R4" V 3780 1600 50  0000 C CNN
+F 0 "R27" V 3780 1600 50  0000 C CNN
 F 1 "120" V 3700 1600 50  0000 C CNN
 F 2 "Resistencias:R_0805" V 3630 1600 50  0001 C CNN
@@
 $EndComp
 $Comp
-L R R6
+L R R28
 U 1 1 5793BE31
 P 3700 1800
-F 0 "R6" V 3780 1800 50  0000 C CNN
+F 0 "R28" V 3780 1800 50  0000 C CNN
 F 1 "120" V 3700 1800 50  0000 C CNN
 F 2 "Resistencias:R_0805" V 3630 1800 50  0001 C CNN
@@
 $EndComp
 $Comp
-L R R3
+L R R32
 U 1 1 5793BE3E
 P 4250 1500
-F 0 "R3" V 4330 1500 50  0000 C CNN
+F 0 "R32" V 4330 1500 50  0000 C CNN
 F 1 "120" V 4250 1500 50  0000 C CNN
 F 2 "Resistencias:R_0805" V 4180 1500 50  0001 C CNN
@@
 $EndComp
 $Comp
-L R R5
+L R R33
 U 1 1 5793BE4B
 P 4250 1700
-F 0 "R5" V 4330 1700 50  0000 C CNN
+F 0 "R33" V 4330 1700 50  0000 C CNN
 F 1 "120" V 4250 1700 50  0000 C CNN
 F 2 "Resistencias:R_0805" V 4180 1700 50  0001 C CNN
@@
 $EndComp
 $Comp
-L R R7
+L R R34
 U 1 1 5793BE58
 P 4250 1900
-F 0 "R7" V 4330 1900 50  0000 C CNN
+F 0 "R34" V 4330 1900 50  0000 C CNN
 F 1 "120" V 4250 1900 50  0000 C CNN
 F 2 "Resistencias:R_0805" V 4180 1900 50  0001 C CNN
@@
 $EndComp
 $Comp
-L R R8
+L R R21
 U 1 1 5793BE65
 P 3250 3100
-F 0 "R8" V 3150 3100 50  0000 C CNN
+F 0 "R21" V 3150 3100 50  0000 C CNN
 F 1 "1K" V 3250 3100 50  0000 C CNN
 F 2 "Resistencias:R_0805" V 3180 3100 50  0001 C CNN
@@
 $EndComp
 $Comp
-L R R9
+L R R22
 U 1 1 5793BE72
 P 3250 3600
-F 0 "R9" V 3150 3600 50  0000 C CNN
+F 0 "R22" V 3150 3600 50  0000 C CNN
 F 1 "1K" V 3250 3600 50  0000 C CNN
 F 2 "Resistencias:R_0805" V 3180 3600 50  0001 C CNN
@@
 $EndComp
 $Comp
-L R R10
+L R R23
 U 1 1 5793BE7F
 P 3250 4100
-F 0 "R10" V 3150 4100 50  0000 C CNN
+F 0 "R23" V 3150 4100 50  0000 C CNN
 F 1 "1K" V 3250 4100 50  0000 C CNN
 F 2 "Resistencias:R_0805" V 3180 4100 50  0001 C CNN
@@
 $EndComp
 $Comp
-L R R12
+L R R25
 U 1 1 5793BE99
 P 3250 5100
-F 0 "R12" V 3150 5100 50  0000 C CNN
+F 0 "R25" V 3150 5100 50  0000 C CNN
 F 1 "1K" V 3250 5100 50  0000 C CNN
 F 2 "Resistencias:R_0805" V 3180 5100 50  0001 C CNN
@@
 	8550 2800 8050 2800
 $Comp
-L BC849 Q1
+L BC849 Q5
 U 1 1 5797F26B
 P 4200 3100
-F 0 "Q1" H 4391 3146 50  0000 L CNN
+F 0 "Q5" H 4391 3146 50  0000 L CNN
 F 1 "SMBT3904" H 4391 3055 50  0000 L CNN
 F 2 "TO_SOT_Packages_SMD:SOT-23" H 4391 3009 50  0001 L CIN
@@
 $EndComp
 $Comp
-L BC849 Q2
+L BC849 Q6
 U 1 1 5797F59C
 P 4600 3600
-F 0 "Q2" H 4791 3646 50  0000 L CNN
+F 0 "Q6" H 4791 3646 50  0000 L CNN
 F 1 "SMBT3904" H 4791 3555 50  0000 L CNN
 F 2 "TO_SOT_Packages_SMD:SOT-23" H 4791 3509 50  0001 L CIN
@@
 $EndComp
 $Comp
-L BC849 Q3
+L BC849 Q7
 U 1 1 5797F60D
 P 5000 4100
-F 0 "Q3" H 5191 4146 50  0000 L CNN
+F 0 "Q7" H 5191 4146 50  0000 L CNN
 F 1 "SMBT3904" H 5191 4055 50  0000 L CNN
 F 2 "TO_SOT_Packages_SMD:SOT-23" H 5191 4009 50  0001 L CIN
@@
 $EndComp
 $Comp
-L BC849 Q4
+L BC849 Q8
 U 1 1 5797F681
 P 5400 4600
-F 0 "Q4" H 5591 4646 50  0000 L CNN
+F 0 "Q8" H 5591 4646 50  0000 L CNN
 F 1 "SMBT3904" H 5591 4555 50  0000 L CNN
 F 2 "TO_SOT_Packages_SMD:SOT-23" H 5591 4509 50  0001 L CIN
@@
 $EndComp
 $Comp
-L BC849 Q5
+L BC849 Q9
 U 1 1 5797F6F8
 P 5800 5100
-F 0 "Q5" H 5991 5146 50  0000 L CNN
+F 0 "Q9" H 5991 5146 50  0000 L CNN
 F 1 "SMBT3904" H 5991 5055 50  0000 L CNN
 F 2 "TO_SOT_Packages_SMD:SOT-23" H 5991 5009 50  0001 L CIN
@@
 $EndBitmap
 $Comp
-L Matriz_5x7_Anodo_Filas U?
+L Matriz_5x7_Anodo_Filas U10
 U 1 1 583F289B
 P 5500 2350
-F 0 "U?" H 5150 2500 60  0000 L CNN
+F 0 "U10" H 5150 2500 60  0000 L CNN
 F 1 "Matriz_5x7_Anodo_Filas" H 5050 3700 60  0000 L CNN
-F 2 "" H 5590 3490 60  0000 C CNN
+F 2 "" H 5590 3490 60  0001 C CNN
 F 3 "" H 5590 3490 60  0000 C CNN
 	1    5500 2350
@@
 $EndComp
 $Comp
-L R R?
+L R R30
 U 1 1 587C05F0
 P 4150 3850
-F 0 "R?" V 4150 3800 50  0000 L CNN
+F 0 "R30" V 4150 3800 50  0000 L CNN
 F 1 "47K" H 3950 3800 50  0000 L CNN
-F 2 "" V 4080 3850 50  0000 C CNN
+F 2 "" V 4080 3850 50  0001 C CNN
 F 3 "" H 4150 3850 50  0000 C CNN
 F 4 "~" H 4150 3850 60  0001 C CNN "Fabricante"
@@
 	4300 3300 4300 6300
 $Comp
-L R R11
+L R R24
 U 1 1 5793BE8C
 P 3250 4600
-F 0 "R11" V 3150 4600 50  0000 C CNN
+F 0 "R24" V 3150 4600 50  0000 C CNN
 F 1 "1K" V 3250 4600 50  0000 C CNN
 F 2 "Resistencias:R_0805" V 3180 4600 50  0001 C CNN
@@
 Connection ~ 4150 3600
 $Comp
-L R R?
+L R R29
 U 1 1 587C2476
 P 3750 3350
-F 0 "R?" V 3750 3300 50  0000 L CNN
+F 0 "R29" V 3750 3300 50  0000 L CNN
 F 1 "47K" H 3550 3300 50  0000 L CNN
-F 2 "" V 3680 3350 50  0000 C CNN
+F 2 "" V 3680 3350 50  0001 C CNN
 F 3 "" H 3750 3350 50  0000 C CNN
 F 4 "~" H 3750 3350 60  0001 C CNN "Fabricante"
@@
 $EndComp
 $Comp
-L R R?
+L R R35
 U 1 1 587C24F4
 P 4500 4350
-F 0 "R?" V 4500 4300 50  0000 L CNN
+F 0 "R35" V 4500 4300 50  0000 L CNN
 F 1 "47K" H 4300 4300 50  0000 L CNN
-F 2 "" V 4430 4350 50  0000 C CNN
+F 2 "" V 4430 4350 50  0001 C CNN
 F 3 "" H 4500 4350 50  0000 C CNN
 F 4 "~" H 4500 4350 60  0001 C CNN "Fabricante"
@@
 $EndComp
 $Comp
-L R R?
+L R R36
 U 1 1 587C258D
 P 4900 4850
-F 0 "R?" V 4900 4800 50  0000 L CNN
+F 0 "R36" V 4900 4800 50  0000 L CNN
 F 1 "47K" H 4700 4800 50  0000 L CNN
-F 2 "" V 4830 4850 50  0000 C CNN
+F 2 "" V 4830 4850 50  0001 C CNN
 F 3 "" H 4900 4850 50  0000 C CNN
 F 4 "~" H 4900 4850 60  0001 C CNN "Fabricante"
@@
 $EndComp
 $Comp
-L R R?
+L R R37
 U 1 1 587C2611
 P 5300 5350
-F 0 "R?" V 5300 5300 50  0000 L CNN
+F 0 "R37" V 5300 5300 50  0000 L CNN
 F 1 "47K" H 5100 5300 50  0000 L CNN
-F 2 "" V 5230 5350 50  0000 C CNN
+F 2 "" V 5230 5350 50  0001 C CNN
 F 3 "" H 5300 5350 50  0000 C CNN
 F 4 "~" H 5300 5350 60  0001 C CNN "Fabricante"

Commit message: asignacion inicial de huellas
Parts:
- R29, R30, R35, R36, R37: footprint (none) -> Resistencias:R_0805
- U10: footprint (none) -> Leds:Matriz_Led_7X5
Changed lines of the file:
@@
 $EndDescr
 $Comp
-L GND #PWR66
+L GND #PWR080
 U 1 1 5793BD55
 P 5100 6550
-F 0 "#PWR66" H 5100 6300 50  0001 C CNN
+F 0 "#PWR080" H 5100 6300 50  0001 C CNN
 F 1 "GND" H 5100 6400 50  0000 C CNN
 F 2 "" H 5100 6550 50  0000 C CNN
@@
 F 0 "U10" H 5150 2500 60  0000 L CNN
 F 1 "Matriz_5x7_Anodo_Filas" H 5050 3700 60  0000 L CNN
-F 2 "" H 5590 3490 60  0001 C CNN
+F 2 "Leds:Matriz_Led_7X5" H 5590 3490 60  0001 C CNN
 F 3 "" H 5590 3490 60  0000 C CNN
 	1    5500 2350
@@
 F 0 "R30" V 4150 3800 50  0000 L CNN
 F 1 "47K" H 3950 3800 50  0000 L CNN
-F 2 "" V 4080 3850 50  0001 C CNN
+F 2 "Resistencias:R_0805" V 4080 3850 50  0001 C CNN
 F 3 "" H 4150 3850 50  0000 C CNN
 F 4 "~" H 4150 3850 60  0001 C CNN "Fabricante"
@@
 F 0 "R29" V 3750 3300 50  0000 L CNN
 F 1 "47K" H 3550 3300 50  0000 L CNN
-F 2 "" V 3680 3350 50  0001 C CNN
+F 2 "Resistencias:R_0805" V 3680 3350 50  0001 C CNN
 F 3 "" H 3750 3350 50  0000 C CNN
 F 4 "~" H 3750 3350 60  0001 C CNN "Fabricante"
@@
 F 0 "R35" V 4500 4300 50  0000 L CNN
 F 1 "47K" H 4300 4300 50  0000 L CNN
-F 2 "" V 4430 4350 50  0001 C CNN
+F 2 "Resistencias:R_0805" V 4430 4350 50  0001 C CNN
 F 3 "" H 4500 4350 50  0000 C CNN
 F 4 "~" H 4500 4350 60  0001 C CNN "Fabricante"
@@
 F 0 "R36" V 4900 4800 50  0000 L CNN
 F 1 "47K" H 4700 4800 50  0000 L CNN
-F 2 "" V 4830 4850 50  0001 C CNN
+F 2 "Resistencias:R_0805" V 4830 4850 50  0001 C CNN
 F 3 "" H 4900 4850 50  0000 C CNN
 F 4 "~" H 4900 4850 60  0001 C CNN "Fabricante"
@@
 F 0 "R37" V 5300 5300 50  0000 L CNN
 F 1 "47K" H 5100 5300 50  0000 L CNN
-F 2 "" V 5230 5350 50  0001 C CNN
+F 2 "Resistencias:R_0805" V 5230 5350 50  0001 C CNN
 F 3 "" H 5300 5350 50  0000 C CNN
 F 4 "~" H 5300 5350 60  0001 C CNN "Fabricante"
