File: Matriz_Led.sch (KiCad schematic (older format))
At the start: 23 parts, among them Q5 SMBT3904, Q6 SMBT3904, Q7 SMBT3904, Q8 SMBT3904, Q9 SMBT3904, U10 Matriz_5x7_Anodo_Filas

Commit message: actualizadas referencias en componentes y ordenado esquema electrico
Parts:
- R29, R30, R35, R36, R37: Fabricante (none) -> VISHAY; Potencia (none) -> 1/8W; Provedor (none) -> TME; Ref (none) -> CRCW080547K0FKEA; Ref_Proveedor (none) -> CRCW080547K0FKEA; Tolerancia (none) -> 1%
- U10: Fabricante (none) -> LUCKY LIGHT; Provedor (none) -> TME; Ref (none) -> KWM-20571ASB; Ref_Proveedor (none) -> KWM-20571ASB
