File: Expansor_ADC.sch (KiCad schematic (older format))
At the start: 4 parts

Commit message: version preliminar de la etapa de alimentacion
Parts:
- gave numbers to parts that had none: 4
Changed lines of the file:
@@
 LIBS:Sensores
 LIBS:Reles
+LIBS:Reguladores
+LIBS:Transistores
 LIBS:Wifi_PB-cache
 EELAYER 26 0
@@
 $Descr User 8268 5846
 encoding utf-8
-Sheet 6 11
+Sheet 6 15
 Title ""
 Date "2017-01-15"
@@
 $EndDescr
 $Comp
-L MCP3204 U?
+L MCP3204 U8
 U 1 1 587AC1C1
 P 4050 2550
-F 0 "U?" H 3600 2050 50  0000 C CNN
+F 0 "U8" H 3600 2050 50  0000 C CNN
 F 1 "MCP3204" H 4450 2050 50  0000 C CNN
 F 2 "" H 4950 2250 50  0001 C CNN
@@
 	5050 2450 4650 2450
 $Comp
-L GND #PWR049
+L GND #PWR44
 U 1 1 587AC29C
 P 4150 3300
-F 0 "#PWR049" H 4150 3050 50  0001 C CNN
+F 0 "#PWR44" H 4150 3050 50  0001 C CNN
 F 1 "GND" H 4155 3127 50  0000 C CNN
 F 2 "" H 4150 3300 50  0000 C CNN
@@
 	4150 3300 4150 3050
 $Comp
-L GNDA #PWR050
+L GNDA #PWR43
 U 1 1 587AC2B9
 P 3950 3300
-F 0 "#PWR050" H 3950 3050 50  0001 C CNN
+F 0 "#PWR43" H 3950 3050 50  0001 C CNN
 F 1 "GNDA" H 3955 3127 50  0000 C CNN
 F 2 "" H 3950 3300 50  0000 C CNN
@@
 	3950 3300 3950 3050
 $Comp
-L CP1 C?
+L CP1 C20
 U 1 1 587BF8DE
 P 4950 1700
-F 0 "C?" H 5065 1746 50  0000 L CNN
+F 0 "C20" H 5065 1746 50  0000 L CNN
 F 1 "CP1" H 5065 1655 50  0000 L CNN
-F 2 "" H 4950 1700 50  0000 C CNN
+F 2 "" H 4950 1700 50  0001 C CNN
 F 3 "" H 4950 1700 50  0000 C CNN
 	1    4950 1700
@@
 $EndComp
 $Comp
-L C C?
+L C C19
 U 1 1 587BF8E5
 P 4500 1700
-F 0 "C?" H 4615 1746 50  0000 L CNN
+F 0 "C19" H 4615 1746 50  0000 L CNN
 F 1 "C" H 4615 1655 50  0000 L CNN
-F 2 "" H 4538 1550 50  0000 C CNN
+F 2 "" H 4538 1550 50  0001 C CNN
 F 3 "" H 4500 1700 50  0000 C CNN
 	1    4500 1700
@@
 	4950 1300 4950 1550
 $Comp
-L GND #PWR?
+L GND #PWR45
 U 1 1 587BF8EE
 P 4500 1950
-F 0 "#PWR?" H 4500 1700 50  0001 C CNN
+F 0 "#PWR45" H 4500 1700 50  0001 C CNN
 F 1 "GND" H 4505 1777 50  0000 C CNN
 F 2 "" H 4500 1950 50  0000 C CNN
@@
 	4950 1950 4950 1850
 $Comp
-L GND #PWR?
+L GND #PWR47
 U 1 1 587BF8F8
 P 4950 1950
-F 0 "#PWR?" H 4950 1700 50  0001 C CNN
+F 0 "#PWR47" H 4950 1700 50  0001 C CNN
 F 1 "GND" H 4955 1777 50  0000 C CNN
 F 2 "" H 4950 1950 50  0000 C CNN
@@
 	4500 1550 4500 1450
 $Comp
-L +3V3 #PWR?
+L +3V3 #PWR46
 U 1 1 587BFA63
 P 4950 1300
-F 0 "#PWR?" H 4950 1150 50  0001 C CNN
+F 0 "#PWR46" H 4950 1150 50  0001 C CNN
 F 1 "+3V3" H 4965 1473 50  0000 C CNN
 F 2 "" H 4950 1300 50  0000 C CNN
@@
 $EndComp
 $Comp
-L C C?
+L C C18
 U 1 1 587BFA96
 P 3650 1700
-F 0 "C?" H 3765 1746 50  0000 L CNN
+F 0 "C18" H 3765 1746 50  0000 L CNN
 F 1 "C" H 3765 1655 50  0000 L CNN
-F 2 "" H 3688 1550 50  0000 C CNN
+F 2 "" H 3688 1550 50  0001 C CNN
 F 3 "" H 3650 1700 50  0000 C CNN
 	1    3650 1700
@@
 $EndComp
 $Comp
-L GNDA #PWR?
+L GNDA #PWR42
 U 1 1 587BFAEE
 P 3650 1950
-F 0 "#PWR?" H 3650 1700 50  0001 C CNN
+F 0 "#PWR42" H 3650 1700 50  0001 C CNN
 F 1 "GNDA" H 3655 1777 50  0000 C CNN
 F 2 "" H 3650 1950 50  0000 C CNN
@@
 	3950 1450 3950 2150
 $Comp
-L +3V3 #PWR?
+L +3V3 #PWR41
 U 1 1 587BFB50
 P 3650 1300
-F 0 "#PWR?" H 3650 1150 50  0001 C CNN
+F 0 "#PWR41" H 3650 1150 50  0001 C CNN
 F 1 "+3V3" H 3665 1473 50  0000 C CNN
 F 2 "" H 3650 1300 50  0000 C CNN

Commit message: asignacion inicial de huellas
Parts:
- C18, C19: value C -> 100n; footprint (none) -> Capacitors_SMD:C_0805
- C20: value CP1 -> 4,7u; footprint (none) -> Capacitors_SMD:C_1206
- U8: footprint (none) -> Housings_SOIC:SOIC-14_3.9x8.7mm_Pitch1.27mm
Connections:
- net CH0: now reaches U8.1 (CH0)
- net CH1: now reaches U8.2 (CH1)
- net CH2: now reaches U8.3 (CH2)
- net CH3: now reaches U8.4 (CH3)
Changed lines of the file:
@@
 F 0 "U8" H 3600 2050 50  0000 C CNN
 F 1 "MCP3204" H 4450 2050 50  0000 C CNN
-F 2 "" H 4950 2250 50  0001 C CNN
+F 2 "Housings_SOIC:SOIC-14_3.9x8.7mm_Pitch1.27mm" H 4950 2250 50  0001 C CNN
 F 3 "" H 4950 2250 50  0001 C CNN
 	1    4050 2550
@@
 	5050 2450 4650 2450
 $Comp
-L GND #PWR44
+L GND #PWR055
 U 1 1 587AC29C
 P 4150 3300
-F 0 "#PWR44" H 4150 3050 50  0001 C CNN
+F 0 "#PWR055" H 4150 3050 50  0001 C CNN
 F 1 "GND" H 4155 3127 50  0000 C CNN
 F 2 "" H 4150 3300 50  0000 C CNN
@@
 	4150 3300 4150 3050
 $Comp
-L GNDA #PWR43
+L GNDA #PWR056
 U 1 1 587AC2B9
 P 3950 3300
-F 0 "#PWR43" H 3950 3050 50  0001 C CNN
+F 0 "#PWR056" H 3950 3050 50  0001 C CNN
 F 1 "GNDA" H 3955 3127 50  0000 C CNN
 F 2 "" H 3950 3300 50  0000 C CNN
@@
 P 4950 1700
 F 0 "C20" H 5065 1746 50  0000 L CNN
-F 1 "CP1" H 5065 1655 50  0000 L CNN
-F 2 "" H 4950 1700 50  0001 C CNN
+F 1 "4,7u" H 5065 1655 50  0000 L CNN
+F 2 "Capacitors_SMD:C_1206" H 4950 1700 50  0001 C CNN
 F 3 "" H 4950 1700 50  0000 C CNN
 	1    4950 1700
@@
 P 4500 1700
 F 0 "C19" H 4615 1746 50  0000 L CNN
-F 1 "C" H 4615 1655 50  0000 L CNN
-F 2 "" H 4538 1550 50  0001 C CNN
+F 1 "100n" H 4615 1655 50  0000 L CNN
+F 2 "Capacitors_SMD:C_0805" H 4538 1550 50  0001 C CNN
 F 3 "" H 4500 1700 50  0000 C CNN
 	1    4500 1700
@@
 	4950 1300 4950 1550
 $Comp
-L GND #PWR45
+L GND #PWR057
 U 1 1 587BF8EE
 P 4500 1950
-F 0 "#PWR45" H 4500 1700 50  0001 C CNN
+F 0 "#PWR057" H 4500 1700 50  0001 C CNN
 F 1 "GND" H 4505 1777 50  0000 C CNN
 F 2 "" H 4500 1950 50  0000 C CNN
@@
 	4950 1950 4950 1850
 $Comp
-L GND #PWR47
+L GND #PWR058
 U 1 1 587BF8F8
 P 4950 1950
-F 0 "#PWR47" H 4950 1700 50  0001 C CNN
+F 0 "#PWR058" H 4950 1700 50  0001 C CNN
 F 1 "GND" H 4955 1777 50  0000 C CNN
 F 2 "" H 4950 1950 50  0000 C CNN
@@
 	4500 1550 4500 1450
 $Comp
-L +3V3 #PWR46
+L +3V3 #PWR059
 U 1 1 587BFA63
 P 4950 1300
-F 0 "#PWR46" H 4950 1150 50  0001 C CNN
+F 0 "#PWR059" H 4950 1150 50  0001 C CNN
 F 1 "+3V3" H 4965 1473 50  0000 C CNN
 F 2 "" H 4950 1300 50  0000 C CNN
@@
 U 1 1 587BFA96
 P 3650 1700
-F 0 "C18" H 3765 1746 50  0000 L CNN
-F 1 "C" H 3765 1655 50  0000 L CNN
-F 2 "" H 3688 1550 50  0001 C CNN
+F 0 "C18" H 3350 1750 50  0000 L CNN
+F 1 "100n" H 3350 1650 50  0000 L CNN
+F 2 "Capacitors_SMD:C_0805" H 3688 1550 50  0001 C CNN
 F 3 "" H 3650 1700 50  0000 C CNN
 	1    3650 1700
@@
 $EndComp
 $Comp
-L GNDA #PWR42
+L GNDA #PWR060
 U 1 1 587BFAEE
 P 3650 1950
-F 0 "#PWR42" H 3650 1700 50  0001 C CNN
+F 0 "#PWR060" H 3650 1700 50  0001 C CNN
 F 1 "GNDA" H 3655 1777 50  0000 C CNN
 F 2 "" H 3650 1950 50  0000 C CNN
@@
 	3950 1450 3950 2150
 $Comp
-L +3V3 #PWR41
+L +3V3 #PWR061
 U 1 1 587BFB50
 P 3650 1300
-F 0 "#PWR41" H 3650 1150 50  0001 C CNN
+F 0 "#PWR061" H 3650 1150 50  0001 C CNN
 F 1 "+3V3" H 3665 1473 50  0000 C CNN
 F 2 "" H 3650 1300 50  0000 C CNN
@@
 $EndComp
 Connection ~ 3650 1450
+Text GLabel 2850 2450 0    60   Input ~ 0
+CH0
+Text GLabel 2850 2550 0    60   Input ~ 0
+CH1
+Text GLabel 2850 2650 0    60   Input ~ 0
+CH2
+Text GLabel 2850 2750 0    60   Input ~ 0
+CH3
+Wire Wire Line
+	2850 2750 3450 2750
+Wire Wire Line
+	3450 2650 2850 2650
+Wire Wire Line
+	2850 2550 3450 2550
+Wire Wire Line
+	3450 2450 2850 2450
 $EndSCHEMATC

Commit message: cambiar ch340T por ch340g y añadir nc a pines
Connections:
- net CLK renamed SCK
- no-connect marks 0 -> 3
Changed lines of the file:
@@
 $Descr User 8268 5846
 encoding utf-8
-Sheet 6 15
+Sheet 6 14
 Title ""
 Date "2017-01-15"
@@
 	5050 2750 4650 2750
 Text GLabel 5050 2450 2    60   Input ~ 0
-CLK
+SCK
 Wire Wire Line
 	5050 2450 4650 2450
 $Comp
-L GND #PWR055
+L GND #PWR063
 U 1 1 587AC29C
 P 4150 3300
-F 0 "#PWR055" H 4150 3050 50  0001 C CNN
+F 0 "#PWR063" H 4150 3050 50  0001 C CNN
 F 1 "GND" H 4155 3127 50  0000 C CNN
 F 2 "" H 4150 3300 50  0000 C CNN
@@
 	4150 3300 4150 3050
 $Comp
-L GNDA #PWR056
+L GNDA #PWR064
 U 1 1 587AC2B9
 P 3950 3300
-F 0 "#PWR056" H 3950 3050 50  0001 C CNN
+F 0 "#PWR064" H 3950 3050 50  0001 C CNN
 F 1 "GNDA" H 3955 3127 50  0000 C CNN
 F 2 "" H 3950 3300 50  0000 C CNN
@@
 	4950 1300 4950 1550
 $Comp
-L GND #PWR057
+L GND #PWR065
 U 1 1 587BF8EE
 P 4500 1950
-F 0 "#PWR057" H 4500 1700 50  0001 C CNN
+F 0 "#PWR065" H 4500 1700 50  0001 C CNN
 F 1 "GND" H 4505 1777 50  0000 C CNN
 F 2 "" H 4500 1950 50  0000 C CNN
@@
 	4950 1950 4950 1850
 $Comp
-L GND #PWR058
+L GND #PWR066
 U 1 1 587BF8F8
 P 4950 1950
-F 0 "#PWR058" H 4950 1700 50  0001 C CNN
+F 0 "#PWR066" H 4950 1700 50  0001 C CNN
 F 1 "GND" H 4955 1777 50  0000 C CNN
 F 2 "" H 4950 1950 50  0000 C CNN
@@
 	4500 1550 4500 1450
 $Comp
-L +3V3 #PWR059
+L +3V3 #PWR067
 U 1 1 587BFA63
 P 4950 1300
-F 0 "#PWR059" H 4950 1150 50  0001 C CNN
+F 0 "#PWR067" H 4950 1150 50  0001 C CNN
 F 1 "+3V3" H 4965 1473 50  0000 C CNN
 F 2 "" H 4950 1300 50  0000 C CNN
@@
 $EndComp
 $Comp
-L GNDA #PWR060
+L GNDA #PWR068
 U 1 1 587BFAEE
 P 3650 1950
-F 0 "#PWR060" H 3650 1700 50  0001 C CNN
+F 0 "#PWR068" H 3650 1700 50  0001 C CNN
 F 1 "GNDA" H 3655 1777 50  0000 C CNN
 F 2 "" H 3650 1950 50  0000 C CNN
@@
 	3950 1450 3950 2150
 $Comp
-L +3V3 #PWR061
+L +3V3 #PWR069
 U 1 1 587BFB50
 P 3650 1300
-F 0 "#PWR061" H 3650 1150 50  0001 C CNN
+F 0 "#PWR069" H 3650 1150 50  0001 C CNN
 F 1 "+3V3" H 3665 1473 50  0000 C CNN
 F 2 "" H 3650 1300 50  0000 C CNN
@@
 Wire Wire Line
 	3450 2450 2850 2450
+NoConn ~ 3450 2550
+NoConn ~ 3450 2650
+NoConn ~ 3450 2750
 $EndSCHEMATC

Commit message: conectar reset gpio. retocar plano masa
Parts:
- added R72: 47K, Resistencias:R_0805, symbol R
Connections:
- net GND: now also R72.2
- net AD_NSS: no longer names the net of U8.8 (~CS)
- net AD_NSS: now also R72.1
- net CH1: no longer names the net of U8.2 (CH1)
- net CH3: no longer names the net of U8.4 (CH3)
- no-connect marks 3 -> 2
Changed lines of the file:
@@
 Wire Wire Line
 	5050 2650 4650 2650
-Text GLabel 5050 2750 2    60   Input ~ 0
-AD_NSS
 Wire Wire Line
-	5050 2750 4650 2750
+	4650 2750 5150 2750
 Text GLabel 5050 2450 2    60   Input ~ 0
 SCK
@@
 	5050 2450 4650 2450
 $Comp
-L GND #PWR062
+L GND #PWR063
 U 1 1 587AC29C
 P 4150 3300
-F 0 "#PWR062" H 4150 3050 50  0001 C CNN
+F 0 "#PWR063" H 4150 3050 50  0001 C CNN
 F 1 "GND" H 4155 3127 50  0000 C CNN
 F 2 "" H 4150 3300 50  0000 C CNN
@@
 	4150 3300 4150 3050
 $Comp
-L GNDA #PWR063
+L GNDA #PWR064
 U 1 1 587AC2B9
 P 3950 3300
-F 0 "#PWR063" H 3950 3050 50  0001 C CNN
+F 0 "#PWR064" H 3950 3050 50  0001 C CNN
 F 1 "GNDA" H 3955 3127 50  0000 C CNN
 F 2 "" H 3950 3300 50  0000 C CNN
@@
 	4950 1300 4950 1550
 $Comp
-L GND #PWR064
+L GND #PWR065
 U 1 1 587BF8EE
 P 4500 1950
-F 0 "#PWR064" H 4500 1700 50  0001 C CNN
+F 0 "#PWR065" H 4500 1700 50  0001 C CNN
 F 1 "GND" H 4505 1777 50  0000 C CNN
 F 2 "" H 4500 1950 50  0000 C CNN
@@
 	4950 1950 4950 1850
 $Comp
-L GND #PWR065
+L GND #PWR066
 U 1 1 587BF8F8
 P 4950 1950
-F 0 "#PWR065" H 4950 1700 50  0001 C CNN
+F 0 "#PWR066" H 4950 1700 50  0001 C CNN
 F 1 "GND" H 4955 1777 50  0000 C CNN
 F 2 "" H 4950 1950 50  0000 C CNN
@@
 	4500 1550 4500 1450
 $Comp
-L +3V3 #PWR066
+L +3V3 #PWR067
 U 1 1 587BFA63
 P 4950 1300
-F 0 "#PWR066" H 4950 1150 50  0001 C CNN
+F 0 "#PWR067" H 4950 1150 50  0001 C CNN
 F 1 "+3V3" H 4965 1473 50  0000 C CNN
 F 2 "" H 4950 1300 50  0000 C CNN
@@
 $EndComp
 $Comp
-L GNDA #PWR067
+L GNDA #PWR068
 U 1 1 587BFAEE
 P 3650 1950
-F 0 "#PWR067" H 3650 1700 50  0001 C CNN
+F 0 "#PWR068" H 3650 1700 50  0001 C CNN
 F 1 "GNDA" H 3655 1777 50  0000 C CNN
 F 2 "" H 3650 1950 50  0000 C CNN
@@
 	3950 1450 3950 2150
 $Comp
-L +3V3 #PWR068
+L +3V3 #PWR069
 U 1 1 587BFB50
 P 3650 1300
-F 0 "#PWR068" H 3650 1150 50  0001 C CNN
+F 0 "#PWR069" H 3650 1150 50  0001 C CNN
 F 1 "+3V3" H 3665 1473 50  0000 C CNN
 F 2 "" H 3650 1300 50  0000 C CNN
@@
 Text GLabel 2850 2450 0    60   Input ~ 0
 CH0
-Text GLabel 2850 2550 0    60   Input ~ 0
-CH1
 Text GLabel 2850 2650 0    60   Input ~ 0
 CH2
-Text GLabel 2850 2750 0    60   Input ~ 0
-CH3
-Wire Wire Line
-	2850 2750 3450 2750
 Wire Wire Line
 	3450 2650 2850 2650
 Wire Wire Line
-	2850 2550 3450 2550
-Wire Wire Line
 	3450 2450 2850 2450
 NoConn ~ 3450 2550
-NoConn ~ 3450 2650
 NoConn ~ 3450 2750
+$Comp
+L GND #PWR070
+U 1 1 58A0F1AC
+P 5150 3300
+F 0 "#PWR070" H 5150 3050 50  0001 C CNN
+F 1 "GND" H 5155 3127 50  0000 C CNN
+F 2 "" H 5150 3300 50  0000 C CNN
+F 3 "" H 5150 3300 50  0000 C CNN
+	1    5150 3300
+	1    0    0    -1
+$EndComp
+Wire Wire Line
+	5150 3300 5150 3200
+Wire Wire Line
+	5150 2750 5150 2900
+$Comp
+L R R72
+U 1 1 58A0F7D5
+P 5150 3050
+F 0 "R72" V 5150 3000 50  0000 L CNN
+F 1 "47K" H 4950 3000 50  0000 L CNN
+F 2 "Resistencias:R_0805" V 5080 3050 50  0001 C CNN
+F 3 "" H 5150 3050 50  0000 C CNN
+F 4 "~" H 5150 3050 60  0001 C CNN "Fabricante"
+F 5 "~" H 5150 3050 60  0001 C CNN "Ref"
+F 6 "~" H 5150 3050 60  0001 C CNN "Potencia"
+F 7 "~" H 5150 3050 60  0001 C CNN "Tolerancia"
+F 8 "~" H 5150 3050 60  0001 C CNN "Provedor"
+F 9 "~" H 5150 3050 60  0001 C CNN "Ref_Proveedor"
+	1    5150 3050
+	1    0    0    -1
+$EndComp
 $EndSCHEMATC
