File: Expansor_ADC.sch (KiCad schematic (older format))
At the start: 5 parts, among them U8 MCP3204

Commit message: actualizadas referencias en componentes y ordenado esquema electrico
Parts:
- C18, C19: Fabricante (none) -> SAMSUNG; Provedor (none) -> TME; Ref (none) -> CL21B104KBCNNNC; Ref_Proveedor (none) -> CL21B104KBCNNNC
- C20: value 4,7u -> 4u7; Fabricante (none) -> SAMSUNG; Provedor (none) -> TME; Ref (none) -> CL31F475ZOFNNNE; Ref_Proveedor (none) -> CL31F475ZOFNNNE
- R72: Fabricante (none) -> VISHAY; Potencia (none) -> 1/8W; Provedor (none) -> TME; Ref (none) -> CRCW080547K0FKEA; Ref_Proveedor (none) -> CRCW080547K0FKEA; Tolerancia (none) -> 1%
- U8: Fabricante (none) -> MICROCHIP TECHNOLOGY; Provedor (none) -> TME; Ref (none) -> MCP3204-CI/SL; Ref_Proveedor (none) -> MCP3204-CI/SL

Commit message: cambiado el driver led al PCA9634
Parts:
- U8: symbol MCP3204 -> MCP3204-RESCUE-Wifi_PB
Changed lines of the file:
@@
 EESchema Schematic File Version 2
+LIBS:Wifi_PB-rescue
 LIBS:power
 LIBS:device
@@
 $EndDescr
 $Comp
-L MCP3204 U8
+L MCP3204-RESCUE-Wifi_PB U8
 U 1 1 587AC1C1
 P 4050 2550
