File: Acelerometro.sch (KiCad schematic (older format))
At the start: 9 parts, among them Q3 BSS138, Q4 BSS138, U5 MMA7660FC

Commit message: cambiado el driver led al PCA9634
Parts:
- Q3, Q4: symbol BSS138 -> BSS138-RESCUE-Wifi_PB
Changed lines of the file:
@@
 EESchema Schematic File Version 2
+LIBS:Wifi_PB-rescue
 LIBS:power
 LIBS:device
@@
 $EndDescr
 $Comp
-L BSS138 Q3
+L BSS138-RESCUE-Wifi_PB Q3
 U 1 1 57952913
 P 5250 2100
+AR Path="/57952913" Ref="Q3"  Part="1"
+AR Path="/587C6740/57952913" Ref="Q3"  Part="1"
 F 0 "Q3" V 5486 2100 50  0000 C CNN
 F 1 "BSS138" V 5577 2100 50  0000 C CNN
@@
 SCL2
 $Comp
-L BSS138 Q4
+L BSS138-RESCUE-Wifi_PB Q4
 U 1 1 57952D65
 P 5900 2600
+AR Path="/57952D65" Ref="Q4"  Part="1"
+AR Path="/587C6740/57952D65" Ref="Q4"  Part="1"
 F 0 "Q4" V 6136 2600 50  0000 C CNN
 F 1 "BSS138" V 6227 2600 50  0000 C CNN
