File: Alimentacion.sch (KiCad schematic (older format))
At the start: 22 parts, among them P1 CONN_01X02, Q10 BC849, Q11 NX2301P, U1 MCP73831T, U12 MCP1640, U2 LD1117S33TR

Commit message: añadidos valores y referencias a control, alimentacion y gpioEx
Parts:
- C1, C4: value 4,7u -> 4u7; Fabricante (none) -> SAMSUNG; Provedor (none) -> TME; Ref (none) -> CL31F475ZOFNNNE; Ref_Proveedor (none) -> CL31F475ZOFNNNE
- C2: Fabricante (none) -> SAMSUNG; Provedor (none) -> TME; Ref (none) -> CL21B104KBCNNNC; Ref_Proveedor (none) -> CL21B104KBCNNNC
- C3, C35: Fabricante (none) -> SAMSUNG; Provedor (none) -> TME; Ref (none) -> CL31B103KBCNNNC; Ref_Proveedor (none) -> CL31B103KBCNNNC
- C34: Fabricante (none) -> SAMSUNG; Provedor (none) -> TME; Ref (none) -> CL31F475ZOFNNNE; Ref_Proveedor (none) -> CL31F475ZOFNNNE
- D1: Fabricante (none) -> OPTOSUPPLY; Provedor (none) -> TME; Ref (none) -> OSR50805C1E; Ref_Proveedor (none) -> OSR50805C1E
- L2: Fabricante (none) -> Bourns; Provedor (none) -> RS; Ref (none) -> SRN4012T-4R7M; Ref_Proveedor (none) -> 850-7445
- P1: Fabricante (none) -> molex; Provedor (none) -> rs; Ref (none) -> 53047-0210; Ref_Proveedor (none) -> 279-9213; Ref_Proveedor 2 (none) -> MX-53047-0210; proveedor 2 (none) -> tme
- Q10: Fabricante (none) -> ON SEMICONDUCTOR; Potencia (none) -> 1/8W; Provedor (none) -> TME; Ref (none) -> BC849CLT1G; Ref_Proveedor (none) -> BC849CLT1G; Tolerancia (none) -> 1%
- Q11: Fabricante (none) -> NXP; Provedor (none) -> TME; Ref (none) -> NX2301P.215; Ref_Proveedor (none) -> NX2301P.215
- R1, R2: Fabricante (none) -> YAGEO; Provedor (none) -> TME; Ref (none) -> RC0805FR-07470RL; Ref_Proveedor (none) -> RC0805FR-07470R; Tolerancia (none) -> 1%
- R54: Fabricante (none) -> VISHAY; Provedor (none) -> TME; Ref (none) -> CRCW08051K00FKEA; Ref_Proveedor (none) -> CRCW08051K00FKEA
- R55: Fabricante (none) -> VISHAY; Potencia (none) -> 1/8W; Provedor (none) -> TME; Ref (none) -> CRCW080547K0FKEA; Ref_Proveedor (none) -> CRCW080547K0FKEA; Tolerancia (none) -> 1%
- R56, R59: Fabricante (none) -> VISHAY; Potencia (none) -> 1/8W; Provedor (none) -> TME; Ref (none) -> CRCW080510K0FKEA; Ref_Proveedor (none) -> CRCW080510K0FKEA; Tolerancia (none) -> 1%
- R57: Fabricante (none) -> Panasonic; Provedor (none) -> RS; Ref (none) -> ERA6AEB9763V; Ref_Proveedor (none) -> 708-7023
- R58: Fabricante (none) -> Panasonic; Provedor (none) -> RS; Ref (none) -> ERA6AEB3093V; Ref_Proveedor (none) -> 708-6871
- U12: Fabricante (none) -> Microchip; Provedor (none) -> RS; Ref (none) -> MCP1640DT-I/CHY; Ref_Proveedor (none) -> 738-6257
Changed lines of the file:
@@
 F 2 "Capacitors_SMD:C_0805" H 8038 2250 50  0001 C CNN
 F 3 "" H 8000 2400 50  0000 C CNN
+F 4 "SAMSUNG" H 7000 1050 60  0001 C CNN "Fabricante"
+F 5 "CL21B104KBCNNNC" H 7000 1050 60  0001 C CNN "Ref"
+F 6 "~" H 7000 1050 60  0001 C CNN "Potencia"
+F 7 "~" H 7000 1050 60  0001 C CNN "Tolerancia"
+F 8 "TME" H 7000 1050 60  0001 C CNN "Provedor"
+F 9 "CL21B104KBCNNNC" H 7000 1050 60  0001 C CNN "Ref_Proveedor"
 	1    8000 2400
 	1    0    0    -1
@@
 F 2 "Capacitors_SMD:C_1206" H 9400 2400 50  0001 C CNN
 F 3 "" H 9400 2400 50  0000 C CNN
+F 4 "SAMSUNG" H 7000 1050 60  0001 C CNN "Fabricante"
+F 5 "CL31B103KBCNNNC" H 7000 1050 60  0001 C CNN "Ref"
+F 6 "~" H 7000 1050 60  0001 C CNN "Potencia"
+F 7 "~" H 7000 1050 60  0001 C CNN "Tolerancia"
+F 8 "TME" H 7000 1050 60  0001 C CNN "Provedor"
+F 9 "CL31B103KBCNNNC" H 7000 1050 60  0001 C CNN "Ref_Proveedor"
 	1    9400 2400
 	1    0    0    -1
@@
 P 2500 2050
 F 0 "C1" H 2615 2096 50  0000 L CNN
-F 1 "4,7u" H 2615 2005 50  0000 L CNN
+F 1 "4u7" H 2615 2005 50  0000 L CNN
 F 2 "Capacitors_SMD:C_1206" H 2538 1900 50  0001 C CNN
 F 3 "" H 2500 2050 50  0001 C CNN
-F 4 "~" H 2500 2050 60  0001 C CNN "Fabricante"
-F 5 "~" H 2500 2050 60  0001 C CNN "Ref"
-F 6 "~" H 2500 2050 60  0001 C CNN "Potencia"
-F 7 "~" H 2500 2050 60  0001 C CNN "Tolerancia"
-F 8 "~" H 2500 2050 60  0001 C CNN "Provedor"
-F 9 "~" H 2500 2050 60  0001 C CNN "Ref_Proveedor"
+F 4 "SAMSUNG" H 1650 1750 60  0001 C CNN "Fabricante"
+F 5 "CL31F475ZOFNNNE" H 1650 1750 60  0001 C CNN "Ref"
+F 6 "~" H 1650 1750 60  0001 C CNN "Potencia"
+F 7 "~" H 1650 1750 60  0001 C CNN "Tolerancia"
+F 8 "TME" H 1650 1750 60  0001 C CNN "Provedor"
+F 9 "CL31F475ZOFNNNE" H 1650 1750 60  0001 C CNN "Ref_Proveedor"
 	1    2500 2050
 	1    0    0    -1
@@
 F 2 "LEDs:LED_0805" H 2850 2050 50  0001 C CNN
 F 3 "" H 2850 2050 50  0001 C CNN
+F 4 "OPTOSUPPLY" H 7000 1050 60  0001 C CNN "Fabricante"
+F 5 "OSR50805C1E" H 7000 1050 60  0001 C CNN "Ref"
+F 6 "~" H 7000 1050 60  0001 C CNN "Potencia"
+F 7 "~" H 7000 1050 60  0001 C CNN "Tolerancia"
+F 8 "TME" H 7000 1050 60  0001 C CNN "Provedor"
+F 9 "OSR50805C1E" H 7000 1050 60  0001 C CNN "Ref_Proveedor"
 	1    2850 2050
 	0    -1   -1   0
@@
 F 2 "Resistencias:R_0805" V 3030 2450 50  0001 C CNN
 F 3 "" H 3100 2450 50  0001 C CNN
+F 4 "YAGEO" H 3100 2450 60  0001 C CNN "Fabricante"
+F 5 "RC0805FR-07470RL" H 3100 2450 60  0001 C CNN "Ref"
+F 6 "~" H 3100 2450 60  0001 C CNN "Potencia"
+F 7 "1%" H 3100 2450 60  0001 C CNN "Tolerancia"
+F 8 "TME" H 3100 2450 60  0001 C CNN "Provedor"
+F 9 "RC0805FR-07470R" H 3100 2450 60  0001 C CNN "Ref_Proveedor"
 	1    3100 2450
 	0    1    1    0
@@
 F 2 "Resistencias:R_0805" V 4580 2150 50  0001 C CNN
 F 3 "" H 4650 2150 50  0001 C CNN
+F 4 "YAGEO" H 3100 2450 60  0001 C CNN "Fabricante"
+F 5 "RC0805FR-07470RL" H 3100 2450 60  0001 C CNN "Ref"
+F 6 "~" H 3100 2450 60  0001 C CNN "Potencia"
+F 7 "1%" H 3100 2450 60  0001 C CNN "Tolerancia"
+F 8 "TME" H 3100 2450 60  0001 C CNN "Provedor"
+F 9 "RC0805FR-07470R" H 3100 2450 60  0001 C CNN "Ref_Proveedor"
 	1    4650 2150
 	0    -1   -1   0
@@
 P 5200 2050
 F 0 "C4" H 5315 2096 50  0000 L CNN
-F 1 "4,7u" H 5315 2005 50  0000 L CNN
+F 1 "4u7" H 5315 2005 50  0000 L CNN
 F 2 "Capacitors_SMD:C_1206" H 5238 1900 50  0001 C CNN
 F 3 "" H 5200 2050 50  0001 C CNN
-F 4 "~" H 5200 2050 60  0001 C CNN "Fabricante"
-F 5 "~" H 5200 2050 60  0001 C CNN "Ref"
-F 6 "~" H 5200 2050 60  0001 C CNN "Potencia"
-F 7 "~" H 5200 2050 60  0001 C CNN "Tolerancia"
-F 8 "~" H 5200 2050 60  0001 C CNN "Provedor"
-F 9 "~" H 5200 2050 60  0001 C CNN "Ref_Proveedor"
+F 4 "SAMSUNG" H 1650 1750 60  0001 C CNN "Fabricante"
+F 5 "CL31F475ZOFNNNE" H 1650 1750 60  0001 C CNN "Ref"
+F 6 "~" H 1650 1750 60  0001 C CNN "Potencia"
+F 7 "~" H 1650 1750 60  0001 C CNN "Tolerancia"
+F 8 "TME" H 1650 1750 60  0001 C CNN "Provedor"
+F 9 "CL31F475ZOFNNNE" H 1650 1750 60  0001 C CNN "Ref_Proveedor"
 	1    5200 2050
 	1    0    0    -1
@@
 F 2 "Connectors_Molex:Molex_PicoBlade_53047-0210_02x1.25mm_Straight" H 5900 1900 50  0001 C CNN
 F 3 "" H 5900 1900 50  0001 C CNN
+F 4 "molex" H 5900 1900 60  0001 C CNN "Fabricante"
+F 5 "53047-0210" H 5900 1900 60  0001 C CNN "Ref"
+F 6 "~" H 5900 1900 60  0001 C CNN "Potencia"
+F 7 "~" H 5900 1900 60  0001 C CNN "Tolerancia"
+F 8 "rs" H 5900 1900 60  0001 C CNN "Provedor"
+F 9 "279-9213" H 5900 1900 60  0001 C CNN "Ref_Proveedor"
+F 10 "tme" H 5900 1900 60  0001 C CNN "proveedor 2"
+F 11 "MX-53047-0210" H 5900 1900 60  0001 C CNN "Ref_Proveedor 2"
 	1    5900 1900
 	1    0    0    -1
@@
 F 2 "TO_SOT_Packages_SMD:SOT-23" H 9000 4125 50  0001 L CNN
 F 3 "" H 8750 4200 50  0001 L CNN
+F 4 "NXP" H 7000 1050 60  0001 C CNN "Fabricante"
+F 5 "NX2301P.215" H 7000 1050 60  0001 C CNN "Ref"
+F 6 "~" H 7000 1050 60  0001 C CNN "Potencia"
+F 7 "~" H 7000 1050 60  0001 C CNN "Tolerancia"
+F 8 "TME" H 7000 1050 60  0001 C CNN "Provedor"
+F 9 "NX2301P.215" H 7000 1050 60  0001 C CNN "Ref_Proveedor"
 	1    8750 4200
 	0    1    -1   0
@@
 F 2 "Resistencias:R_0805" V 8980 4650 50  0001 C CNN
 F 3 "" H 9050 4650 50  0001 C CNN
+F 4 "VISHAY" H 4350 1650 60  0001 C CNN "Fabricante"
+F 5 "CRCW080510K0FKEA" H 4350 1650 60  0001 C CNN "Ref"
+F 6 "1/8W" H 4350 1650 60  0001 C CNN "Potencia"
+F 7 "1%" H 4350 1650 60  0001 C CNN "Tolerancia"
+F 8 "TME" H 4350 1650 60  0001 C CNN "Provedor"
+F 9 "CRCW080510K0FKEA" H 4350 1650 60  0001 C CNN "Ref_Proveedor"
 	1    9050 4650
 	0    1    1    0
@@
 F 2 "TO_SOT_Packages_SMD:SOT-23-6" H 3500 4900 60  0001 C CNN
 F 3 "" H 3500 4900 60  0001 C CNN
+F 4 "Microchip" H 7000 1050 60  0001 C CNN "Fabricante"
+F 5 "MCP1640DT-I/CHY" H 7000 1050 60  0001 C CNN "Ref"
+F 6 "~" H 7000 1050 60  0001 C CNN "Potencia"
+F 7 "~" H 7000 1050 60  0001 C CNN "Tolerancia"
+F 8 "RS" H 7000 1050 60  0001 C CNN "Provedor"
+F 9 "738-6257" H 7000 1050 60  0001 C CNN "Ref_Proveedor"
 	1    3500 4900
 	1    0    0    -1
@@
 F 2 "Magneticos:BOURNS_SRN4012T" H 2950 3600 50  0001 C CNN
 F 3 "" H 2950 3600 50  0001 C CNN
+F 4 "Bourns" H 7000 1050 60  0001 C CNN "Fabricante"
+F 5 "SRN4012T-4R7M" H 7000 1050 60  0001 C CNN "Ref"
+F 6 "~" H 7000 1050 60  0001 C CNN "Potencia"
+F 7 "~" H 7000 1050 60  0001 C CNN "Tolerancia"
+F 8 "RS" H 7000 1050 60  0001 C CNN "Provedor"
+F 9 "850-7445" H 7000 1050 60  0001 C CNN "Ref_Proveedor"
 	1    2950 3600
 	0    -1   -1   0
@@
 F 2 "Capacitors_SMD:C_1206" H 2238 4550 50  0001 C CNN
 F 3 "" H 2200 4700 50  0001 C CNN
+F 4 "SAMSUNG" H 1650 1750 60  0001 C CNN "Fabricante"
+F 5 "CL31F475ZOFNNNE" H 1650 1750 60  0001 C CNN "Ref"
+F 6 "~" H 1650 1750 60  0001 C CNN "Potencia"
+F 7 "~" H 1650 1750 60  0001 C CNN "Tolerancia"
+F 8 "TME" H 1650 1750 60  0001 C CNN "Provedor"
+F 9 "CL31F475ZOFNNNE" H 1650 1750 60  0001 C CNN "Ref_Proveedor"
 	1    2200 4700
 	1    0    0    -1
@@
 F 2 "Resistencias:R_0805" V 4280 4300 50  0001 C CNN
 F 3 "" H 4350 4300 50  0001 C CNN
+F 4 "Panasonic" H 7000 1050 60  0001 C CNN "Fabricante"
+F 5 "ERA6AEB9763V" H 7000 1050 60  0001 C CNN "Ref"
+F 6 "~" H 7000 1050 60  0001 C CNN "Potencia"
+F 7 "~" H 7000 1050 60  0001 C CNN "Tolerancia"
+F 8 "RS" H 7000 1050 60  0001 C CNN "Provedor"
+F 9 "708-7023" H 7000 1050 60  0001 C CNN "Ref_Proveedor"
 	1    4350 4300
 	1    0    0    -1
@@
 F 2 "Resistencias:R_0805" V 4280 4850 50  0001 C CNN
 F 3 "" H 4350 4850 50  0001 C CNN
+F 4 "Panasonic" H 7000 1050 60  0001 C CNN "Fabricante"
+F 5 "ERA6AEB3093V" H 7000 1050 60  0001 C CNN "Ref"
+F 6 "~" H 7000 1050 60  0001 C CNN "Potencia"
+F 7 "~" H 7000 1050 60  0001 C CNN "Tolerancia"
+F 8 "RS" H 7000 1050 60  0001 C CNN "Provedor"
+F 9 "708-6871" H 7000 1050 60  0001 C CNN "Ref_Proveedor"
 	1    4350 4850
 	1    0    0    -1
@@
 F 2 "Capacitors_SMD:C_1206" H 5038 4550 50  0001 C CNN
 F 3 "" H 5000 4700 50  0001 C CNN
+F 4 "SAMSUNG" H 7000 1050 60  0001 C CNN "Fabricante"
+F 5 "CL31B103KBCNNNC" H 7000 1050 60  0001 C CNN "Ref"
+F 6 "~" H 7000 1050 60  0001 C CNN "Potencia"
+F 7 "~" H 7000 1050 60  0001 C CNN "Tolerancia"
+F 8 "TME" H 7000 1050 60  0001 C CNN "Provedor"
+F 9 "CL31B103KBCNNNC" H 7000 1050 60  0001 C CNN "Ref_Proveedor"
 	1    5000 4700
 	1    0    0    -1
@@
 F 2 "TO_SOT_Packages_SMD:SOT-23" H 2850 5675 50  0001 L CIN
 F 3 "" H 2650 5750 50  0001 L CNN
+F 4 "ON SEMICONDUCTOR" H 4350 1650 60  0001 C CNN "Fabricante"
+F 5 "BC849CLT1G" H 4350 1650 60  0001 C CNN "Ref"
+F 6 "1/8W" H 4350 1650 60  0001 C CNN "Potencia"
+F 7 "1%" H 4350 1650 60  0001 C CNN "Tolerancia"
+F 8 "TME" H 4350 1650 60  0001 C CNN "Provedor"
+F 9 "BC849CLT1G" H 4350 1650 60  0001 C CNN "Ref_Proveedor"
 	1    2650 5750
 	1    0    0    -1
@@
 F 2 "Resistencias:R_0805" V 2180 6250 50  0001 C CNN
 F 3 "" H 2250 6250 50  0001 C CNN
+F 4 "VISHAY" H 4350 1650 60  0001 C CNN "Fabricante"
+F 5 "CRCW080547K0FKEA" H 4350 1650 60  0001 C CNN "Ref"
+F 6 "1/8W" H 4350 1650 60  0001 C CNN "Potencia"
+F 7 "1%" H 4350 1650 60  0001 C CNN "Tolerancia"
+F 8 "TME" H 4350 1650 60  0001 C CNN "Provedor"
+F 9 "CRCW080547K0FKEA" H 4350 1650 60  0001 C CNN "Ref_Proveedor"
 	1    2250 6250
 	1    0    0    -1
@@
 F 2 "Resistencias:R_0805" V 2480 4450 50  0001 C CNN
 F 3 "" H 2550 4450 50  0001 C CNN
+F 4 "VISHAY" H 4350 1650 60  0001 C CNN "Fabricante"
+F 5 "CRCW080510K0FKEA" H 4350 1650 60  0001 C CNN "Ref"
+F 6 "1/8W" H 4350 1650 60  0001 C CNN "Potencia"
+F 7 "1%" H 4350 1650 60  0001 C CNN "Tolerancia"
+F 8 "TME" H 4350 1650 60  0001 C CNN "Provedor"
+F 9 "CRCW080510K0FKEA" H 4350 1650 60  0001 C CNN "Ref_Proveedor"
 	1    2550 4450
 	0    1    1    0
@@
 F 2 "Resistencias:R_0805" V 1780 5750 50  0001 C CNN
 F 3 "" H 1850 5750 50  0001 C CNN
+F 4 "VISHAY" H 1650 1750 60  0001 C CNN "Fabricante"
+F 5 "CRCW08051K00FKEA" H 1650 1750 60  0001 C CNN "Ref"
+F 6 "~" H 1650 1750 60  0001 C CNN "Potencia"
+F 7 "~" H 1650 1750 60  0001 C CNN "Tolerancia"
+F 8 "TME" H 1650 1750 60  0001 C CNN "Provedor"
+F 9 "CRCW08051K00FKEA" H 1650 1750 60  0001 C CNN "Ref_Proveedor"
 	1    1850 5750
 	0    1    1    0
