File: LDR.sch (KiCad schematic (older format))
At the start: 2 parts

Commit message: actualizadas referencias en componentes y ordenado esquema electrico
Parts:
- R47: Ref GM7516 -> GM4516; Ref_Proveedor GM7516 -> GM4516
