File: Leds.sch (KiCad schematic (older format))
At the start: 12 parts

Commit message: actualizadas referencias en componentes y ordenado esquema electrico
Parts:
- D4, D5, D6, D7: Fabricante (none) -> OPTOSUPPLY; Provedor (none) -> TME; Ref (none) -> OSR50805C1E; Ref_Proveedor (none) -> OSR50805C1E
- R38, R62, R63, R64: value R -> 220; Fabricante (none) -> YAGEO; Provedor (none) -> TME; Ref (none) -> RC0805FR-07220RL; Ref_Proveedor (none) -> RC0805FR-07220R
