File: Pulsadores.sch (KiCad schematic (older format))
At the start: 25 parts, among them P10 CONN_01X01, P16 CONN_01X01, P17 CONN_01X01, P18 CONN_01X01, P19 CONN_01X01, P6 CONN_01X01, P7 CONN_01X01, P8 CONN_01X01, P9 CONN_01X01, SW1 Pulsador_2p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

Commit message: actualizadas referencias en componentes y ordenado esquema electrico
Parts:
- SW1, SW2, SW3, SW4: Fabricante (none) -> CANAL ELECTRONIC; Provedor (none) -> TME; Ref (none) -> DTSM-31N-B; Ref_Proveedor (none) -> DTSM31NB
